File: DemoGit.kicad_sch (KiCad schematic)
At the start: 17 parts, among them J1 USB_B_Micro, J2 Conn_Coaxial, SW1 SW_Push, U1 AP2112K-3.3, U2 RFM95W-915S2, U3 ATSAMD21G15A-A, U4 Waveshare_epaper

Commit message: fix(bom): cambia R2 a 4.7k
Parts:
- R2: value 10k -> 4.7k
Changed lines of the file:
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@@
 			)
 		)
-		(property "Value" "10k"
+		(property "Value" "4.7k"
 			(at 256.54 99.06 90)
 			(show_name no)
