File: DemoGit.kicad_sch (KiCad schematic)
At the start: 16 parts, among them J1 USB_B_Micro, J2 Conn_Coaxial, SW1 SW_Push, U1 AP2112K-3.3, U2 RFM95W-915S2, U3 ATSAMD21G15A-A

Commit message: feat(sch): agrega display e-ink U4 al esquematico
Parts:
- added U4: Waveshare_epaper, symbol E_Ink_Display:E_ink_display
Connections:
- net 3V3: now also U4.8 (VCC)
- net CLK: now also U4.5 (SPLCLK)
- net COPI: now also U4.6 (SPLDIN)
- net GND: now also U4.7 (GND)

Commit message: fix(bom): cambia R2 a 1k
Parts:
- R2: value 10k -> 1k
Changed lines of the file:
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@@
 			)
 		)
-		(property "Value" "10k"
+		(property "Value" "1k"
 			(at 256.54 99.06 90)
 			(show_name no)
